Commit message: Added casters to Arlo robot URDF model

File: src/activitybot_description/urdf/create.urdf.xacro (robot description, xacro)
@@ -1,5 +1,5 @@
 <?xml version="1.0"?>
 <robot name="turtlebot_hardware" xmlns:xacro="http://ros.org/wiki/xacro">
-  <!-- Macro for TurtleBot body. Including Gazebo extensions, but does not include Kinect -->
+  <!-- Macro for ActivityBot body. -->
   <xacro:include filename="$(find create_description)/urdf/create_gazebo.urdf.xacro"/>
   <property name="base_x" value="0.33" />
@@ -79,4 +79,50 @@
 	    <child link="battery_box" />
 	  </joint>
+	  <link name="front_caster">
+	    <inertial>
+	      <mass value="0.001" />
+	      <origin xyz="0 0 0" />
+	      <inertia ixx="0.0001" ixy="0.0" ixz="0.0"
+	        iyy="0.0001" iyz="0.0"
+	        izz="0.0001" />
+	    </inertial>
+	    <visual>
+	      <origin xyz="0 0 0" rpy="-1.5707 0 1.5707" />
+	      <geometry>
+	        <mesh filename="package://activitybot_description/meshes/28971-Caster-Wheel-Kit-v1.0.stl"/>
+	      </geometry>
+        <material name ="light_grey">
+            <color rgba="0.6 0.6 0.6 1"/>
+        </material>
+	    </visual>
+      </link>
+      <joint name="front_caster_joint" type="fixed">
+	    <origin xyz="0.18745 0 -0.00475" rpy="0 0 0" />
+	    <parent link="base_link" />
+	    <child link="front_caster" />
+	  </joint>
+	  <link name="rear_caster">
+	    <inertial>
+	      <mass value="0.001" />
+	      <origin xyz="0 0 0" />
+	      <inertia ixx="0.0001" ixy="0.0" ixz="0.0"
+	        iyy="0.0001" iyz="0.0"
+	        izz="0.0001" />
+	    </inertial>
+	    <visual>
+	      <origin xyz="0 0 0" rpy="-1.5707 0 1.5707" />
+	      <geometry>
+	        <mesh filename="package://activitybot_description/meshes/28971-Caster-Wheel-Kit-v1.0.stl"/>
+	      </geometry>
+        <material name ="light_grey">
+            <color rgba="0.6 0.6 0.6 1"/>
+        </material>
+	    </visual>
+      </link>
+      <joint name="rear_caster_joint" type="fixed">
+	    <origin xyz="-0.18745 0 -0.00475" rpy="0 0 0" />
+	    <parent link="base_link" />
+	    <child link="rear_caster" />
+	  </joint>
 	  <link name="wall_sensor_link">
 	    <inertial>
