Commit message: Renamed create.urdf.xacro to arlo.urdf.xacro and removed TurtleBot specific items

File: src/activitybot_description/urdf/activitybot.urdf.xacro (robot description, xacro)
@@ -5,10 +5,10 @@
     - 3d Sensor : kinect
 -->
-<robot name="turtlebot" xmlns:xacro="http://ros.org/wiki/xacro">
+<robot name="arlobot" xmlns:xacro="http://ros.org/wiki/xacro">
   <!-- General -->
   <xacro:include filename="$(find turtlebot_description)/urdf/common_properties.urdf.xacro"/>
   <xacro:include filename="$(find turtlebot_description)/urdf/turtlebot_properties.urdf.xacro"/>
   <!-- Bases -->
-  <xacro:include filename="$(find activitybot_description)/urdf/create.urdf.xacro"/>
+  <xacro:include filename="$(find activitybot_description)/urdf/arlo.urdf.xacro"/>
   <!-- Stacks -->
   <xacro:include filename="$(find activitybot_description)/urdf/circles.urdf.xacro"/>

File: src/activitybot_description/urdf/arlo.urdf.xacro (robot description, xacro)
@@ -1,6 +1,5 @@
 <?xml version="1.0"?>
-<robot name="turtlebot_hardware" xmlns:xacro="http://ros.org/wiki/xacro">
+<robot name="arlobot_hardware" xmlns:xacro="http://ros.org/wiki/xacro">
   <!-- Macro for ActivityBot body. -->
-  <xacro:include filename="$(find create_description)/urdf/create_gazebo.urdf.xacro"/>
   <property name="base_x" value="0.33" />
   <property name="base_y" value="0.33" />
@@ -125,73 +124,8 @@
 	    <child link="rear_caster" />
 	  </joint>
-	  <link name="wall_sensor_link">
-	    <inertial>
-	      <mass value="0.01" />
-	      <origin xyz="0 0 0"/>
-	      <inertia ixx="0.001" ixy="0.0" ixz="0.0"
-	        iyy="0.001" iyz="0.0" izz="0.001" />
-	    </inertial>
-	  </link>
-	  <link name="left_cliff_sensor_link">
-	    <inertial>
-	      <mass value="0.01" />
-	      <origin xyz="0 0 0"/>
-	      <inertia ixx="0.001" ixy="0.0" ixz="0.0"
-	        iyy="0.001" iyz="0.0" izz="0.001" />
-	    </inertial>
-	  </link>
-	  <link name="right_cliff_sensor_link">
-	    <inertial>
-	      <mass value="0.01" />
-	      <origin xyz="0 0 0"/>
-	      <inertia ixx="0.001" ixy="0.0" ixz="0.0"
-	        iyy="0.001" iyz="0.0" izz="0.001" />
-	    </inertial>
-	  </link>
-	  <link name="leftfront_cliff_sensor_link">
-	    <inertial>
-	      <mass value="0.01" />
-	      <origin xyz="0 0 0"/>
-	      <inertia ixx="1.0" ixy="0.0" ixz="0.0"
-	        iyy="0.01" iyz="0.0" izz="0.01" />
-	    </inertial>
-	  </link>
-	  <link name="rightfront_cliff_sensor_link">
-	    <inertial>
-	      <mass value="0.01" />
-	      <origin xyz="0 0 0"/>
-	      <inertia ixx="0.001" ixy="0.0" ixz="0.0"
-	        iyy="0.001" iyz="0.0" izz="0.001" />
-	    </inertial>
-	  </link>
 	  <joint name="base_footprint_joint" type="fixed">
 	    <origin xyz="0 0 0.10125" rpy="0 0 0" />
 	    <parent link="base_footprint"/>
 	    <child link="base_link" />
-	  </joint>
-	  <joint name="base_wall_sensor_joint" type="fixed">
-	    <origin xyz="0.09 -0.120 0.042" rpy="0 0 -1.0" />
-	    <parent link="base_link"/>
-	    <child link="wall_sensor_link" />
-	  </joint>
-	  <joint name="base_left_cliff_sensor_joint" type="fixed">
-	    <origin xyz="0.07 0.14 0.01" rpy="0 1.57079 0" />
-	    <parent link="base_link"/>
-	    <child link="left_cliff_sensor_link" />
-	  </joint>
-	  <joint name="base_right_cliff_sensor_joint" type="fixed">
-	    <origin xyz="0.07 -0.14 0.01" rpy="0 1.57079 0" />
-	    <parent link="base_link"/>
-	    <child link="right_cliff_sensor_link" />
-	  </joint>
-	  <joint name="base_leftfront_cliff_sensor_joint" type="fixed">
-	    <origin xyz="0.15 0.04 0.01" rpy="0 1.57079 0" />
-	    <parent link="base_link"/>
-	    <child link="leftfront_cliff_sensor_link" />
-	  </joint>
-	  <joint name="base_rightfront_cliff_sensor_joint" type="fixed">
-	    <origin xyz="0.15 -0.04 0.01" rpy="0 1.57079 0" />
-	    <parent link="base_link"/>
-	    <child link="rightfront_cliff_sensor_link" />
 	  </joint>
 	  <link name="left_axle_link">
@@ -307,71 +241,4 @@
 	    <axis xyz="0 1 0"/>
 	  </joint>
-	  <link name="rear_wheel_link">
-	    <inertial>
-	      <origin xyz="0 0 0"/>
-	      <mass value="0.001" />
-	      <inertia ixx="0.0001" ixy="0.0" ixz="0.0"
-	        iyy="0.0001" iyz="0.0" izz="0.0001" />
-	    </inertial>
-	    <visual>
-	      <origin xyz="0 0 0" rpy="0 1.5707 1.5707"/>
-	      <geometry>
-	        <sphere radius="0.015" />
-	      </geometry>
-	    </visual>
-	    <collision>
-	      <origin xyz="0 0 0" rpy="0 1.5707 1.5707" />
-	      <geometry>
-	        <sphere radius="0.015" />
-	      </geometry>
-	    </collision>
-	  </link>
-	  <!-- fixed because there's no transmission -->
-	  <joint name="rear_castor_joint" type="fixed">
-	    <origin xyz="-0.13 0 0.0" rpy="0 0 0"/>
-	    <parent link="base_link"/>
-	    <child link="rear_wheel_link"/>
-	    <axis xyz="0 1 0"/>
-	  </joint>
-	  <link name="front_wheel_link">
-	    <inertial>
-	      <origin xyz="0 0 0" />
-	      <mass value="0.01" />
-	      <inertia ixx="0.001" ixy="0.0" ixz="0.0"
-	        iyy="0.001" iyz="0.0" izz="0.001" />
-	    </inertial>
-	    <visual>
-	      <origin xyz="0 0 0" rpy="0 1.5707 1.5707"/>
-	      <geometry>
-	        <sphere radius="0.018" />
-	      </geometry>
-	    </visual>
-	    <collision>
-	      <origin xyz="0 0 0" rpy="0 1.5707 1.5707" />
-	      <geometry>
-	        <sphere radius="0.018" />
-	      </geometry>
-	    </collision>
-	  </link>
-	  <!-- fixed because there's no transmission -->
-	  <joint name="front_castor_joint" type="fixed">
-	    <origin xyz="0.13 0 0.0" rpy="0 0 0"/>
-	    <parent link="base_link"/>
-	    <child link="front_wheel_link"/>
-	    <axis xyz="0 1 0"/>
-	  </joint>
-	  <joint name="gyro_joint" type="fixed">
-	    <axis xyz="0 1 0" />
-	    <origin xyz="0 0 0.04" rpy="0 0 0" />
-	    <parent link="base_link"/>
-	    <child link="gyro_link"/>
-	  </joint>
-	  <link name="gyro_link">
-	    <inertial>
-	      <mass value="0.001" />
-	      <origin xyz="0 0 0" rpy="0 0 0" />
-	      <inertia ixx="0.0001" ixy="0" ixz="0" iyy="0.000001" iyz="0" izz="0.0001" />
-	    </inertial>
-	  </link>
 	  <joint name="laser_joint" type="fixed">
 	    <origin xyz="-0.065 0 0.075" rpy="0 0 0" />
@@ -414,9 +281,4 @@
 	    </inertial>
 	  </link>
-	  <!-- Simulation sensors -->
-	  <sim_create/>
-	  <sim_create_wall_sensor/>
-	  <sim_create_cliff_sensors/>
-    <sim_imu/>
   </xacro:macro>
 </robot>

Commit message: Cleaned up URDF files and added some startup scripts

File: src/activitybot_description/urdf/activitybot.urdf.xacro (robot description, xacro)
@@ -1,16 +1,15 @@
 <?xml version="1.0"?>
-<!--
-    - Base      : create
-    - Stacks    : circles
-    - 3d Sensor : kinect
--->
 <robot name="arlobot" xmlns:xacro="http://ros.org/wiki/xacro">
-  <!-- General -->
+  <!-- Various useful properties such as constants and materials from TurtleBot -->
   <xacro:include filename="$(find turtlebot_description)/urdf/common_properties.urdf.xacro"/>
+  <!--
+    These properties must be observed by any machine
+    that wants to be defined as a turtlebot. Refer
+    to the REP for more details.
+    http://www.ros.org/reps/rep-0119.html
+   -->
   <xacro:include filename="$(find turtlebot_description)/urdf/turtlebot_properties.urdf.xacro"/>
-  <!-- Bases -->
+  <!-- ArloBot -->
   <xacro:include filename="$(find activitybot_description)/urdf/arlo.urdf.xacro"/>
-  <!-- Stacks -->
-  <xacro:include filename="$(find activitybot_description)/urdf/circles.urdf.xacro"/>
   <!-- 3D Sensors -->
   <xacro:include filename="$(find turtlebot_description)/urdf/sensors/kinect.urdf.xacro"/>

File: src/activitybot_description/urdf/arlo.urdf.xacro (robot description, xacro)
@@ -282,3 +282,69 @@
 	  </link>
   </xacro:macro>
+  <xacro:macro name="turtlebot_standoff_5in" params="parent number x_loc y_loc z_loc">
+    <joint name="standoff_5in_${number}_joint" type="fixed">
+      <origin xyz="${x_loc} ${y_loc} ${z_loc}" rpy="0 0 0" />
+      <parent link="${parent}"/>
+      <child link="standoff_5in_${number}_link" />
+    </joint>
+    <link name="standoff_5in_${number}_link">
+      <inertial>
+        <mass value="0.001" />
+        <origin xyz="0 0 0" />
+        <inertia ixx="0.0001" ixy="0.0" ixz="0.0"
+          iyy="0.0001" iyz="0.0"
+          izz="0.0001" />
+      </inertial>
+      <visual>
+        <origin xyz=" 0 0 0 " rpy="0 0 0" />
+        <geometry>
+          <cylinder length="0.127" radius="0.00635"/>
+        </geometry>
+        <material name ="light_grey">
+            <color rgba="0.6 0.6 0.6 1"/>
+        </material>
+      </visual>
+      <collision>
+        <origin xyz="0.0 0.0 0.0" rpy="0 0 0" />
+        <geometry>
+          <cylinder length="0.127" radius="0.00635"/>
+        </geometry>
+      </collision>
+    </link>
+  </xacro:macro>
+  <xacro:macro name="stack_circles" params="parent">
+    <joint name="plate_0_joint" type="fixed">
+      <origin xyz="0 0 0.1365" rpy="0 0 0" />
+      <parent link="${parent}"/>
+      <child link="plate_0_link" />
+    </joint>
+    <link name="plate_0_link">
+      <inertial>
+        <mass value="0.01" />
+        <origin xyz="0 0 0" />
+        <inertia ixx="0.01" ixy="0.0" ixz="0.0"
+          iyy="0.01" iyz="0.0"
+          izz="0.01" />
+      </inertial>
+      <visual>
+        <origin xyz=" 0 0 0 " rpy="0 0 0" />
+        <geometry>
+          <cylinder length="0.0095" radius="0.22545"/>
+        </geometry>
+        <material name ="veryDarkGrey">
+            <color rgba=".2 .2 .2 1"/>
+        </material>
+      </visual>
+      <collision>
+        <origin xyz="0.0 0.0 0.0" rpy="0 0 0" />
+        <geometry>
+          <cylinder length="0.0095" radius="0.22545"/>
+        </geometry>
+      </collision>
+    </link>
+    <turtlebot_standoff_5in parent="${parent}" number="0" x_loc="0.0676402" y_loc="0.1314196" z_loc="0.06825"/>
+    <turtlebot_standoff_5in parent="${parent}" number="1" x_loc="0.0676402" y_loc="-0.1314196" z_loc="0.06825"/>
+    <turtlebot_standoff_5in parent="${parent}" number="2" x_loc="-0.052832" y_loc="-0.1314196" z_loc="0.06825"/>
+    <turtlebot_standoff_5in parent="${parent}" number="3" x_loc="-0.052832" y_loc="0.1314196" z_loc="0.06825"/>
+  </xacro:macro>
 </robot>
