Commit message: More URDF cleanup

File: src/activitybot_description/urdf/arlo.urdf.xacro (robot description, xacro)
@@ -241,24 +241,4 @@
 	    <axis xyz="0 1 0"/>
 	  </joint>
-	  <joint name="laser_joint" type="fixed">
-	    <origin xyz="-0.065 0 0.075" rpy="0 0 0" />
-	    <parent link="base_link" />
-	    <child link="laser" />
-	  </joint>
-	  <link name="laser">
-	    <visual>
-	      <geometry>
-	        <box size="0.02 0.035 0.002" />
-	      </geometry>
-	      <material name="Green" />
-	    </visual>
-	    <inertial>
-	      <mass value="0.001" />
-	      <origin xyz="0 0 0" />
-	      <inertia ixx="0.0001" ixy="0.0" ixz="0.0"
-	        iyy="0.0001" iyz="0.0"
-	        izz="0.0001" />
-	    </inertial>
-	  </link>
 	  <joint name="ping_array_joint" type="fixed">
 	    <origin xyz="0.065 0 0.05" rpy="0 0 0" />

Commit message: Updated and improved URDF model

File: src/activitybot_description/urdf/arlo.urdf.xacro (robot description, xacro)
@@ -242,5 +242,5 @@
 	  </joint>
 	  <joint name="ping_array_joint" type="fixed">
-	    <origin xyz="0.065 0 0.05" rpy="0 0 0" />
+	    <origin xyz="0.18745 0 0.03695" rpy="0 0 0" />
 	    <parent link="base_link" />
 	    <child link="ping_sensor_array" />
@@ -249,7 +249,6 @@
 	    <visual>
 	      <geometry>
-	        <box size="0.02 0.035 0.002" />
-	      </geometry>
-	      <material name="Green" />
+	        <box size="0.0174 0.06 0.0644" />
+	      </geometry>
 	    </visual>
 	    <inertial>
